File: KiCad/Ice40hx4k_tq144/Ice40hx4k_tq144.kicad_pcb (KiCad board)
At the start: 2 copper layers, 99.1 x 99.1 mm, 229 parts, among them J1 +5V, J2 +3V3, J21 PROGRAM, J22 USB_B_Micro, J3 SWD, J4 VGA, J9 2354 BOOT SEL, U1 LD1117S33TR_SOT223, U10 74CBTD3861, U11 LSF0108PW, U12 LSF0108PW, U13 LSF0108PW, U14 LSF0108PW, U15 74CBTD3861, U16 iCE40HX4K-TQ144, U18 TLV74311PDBVR, U19 RP2354A-QFN60, U2 MIC5504-1.2YM5, U3 W25Q16JVSSIQ, U5 LSF0108PW, U6 74CBTD3861, U7 74CBTD3861, U8 74CBTD3861, U9 74CBTD3861, Y1 12MHz

Commit message: - Swapped SDI / SDO so i can have a straight through cable to the programmer board.
Parts:
- J4: footprint SamacSys_Parts:117345301 -> _Custom:DSUB-15
Connections:
- J21 pad 2: /iCE40-SDI -> /iCE40-SDO
- J21 pad 3: /iCE40-SDO -> /iCE40-SDI
Routing:
- net /iCE40-SDI: track 45.9 -> 46.9 mm
- net /iCE40-SDO: track 50.1 -> 50.4 mm, vias 0 -> 1
Other:
- board text added: "CLOCK"
- board text added: "DONE"
- board text added: "SDI"
- board text added: "SDO"
- board text added: "~{CS}"
- board text added: "~{RESET}"
