File: KiCad/Ice40hx4k_tq144/Ice40hx4k_tq144.kicad_sch (KiCad schematic)
At the start: 229 parts, among them J1 +5V, J2 +3V3, J21 PROGRAM, J22 USB_B_Micro, J3 SWD, J4 VGA, J9 2354 BOOT SEL, U1 LD1117S33TR_SOT223, U10 74CBTD3861, U11 LSF0108PW, U12 LSF0108PW, U13 LSF0108PW, U14 LSF0108PW, U15 74CBTD3861, U16 iCE40HX4K-TQ144, U18 TLV74311PDBVR, U19 RP2354A-QFN60, U2 MIC5504-1.2YM5, U3 W25Q16JVSSIQ, U5 LSF0108PW, U6 74CBTD3861, U7 74CBTD3861, U8 74CBTD3861, U9 74CBTD3861, Y1 12MHz

Commit message: - Swapped SDI / SDO so i can have a straight through cable to the programmer board.
Parts:
- J4: footprint SamacSys_Parts:117345301 -> _Custom:DSUB-15; symbol Connector:DE15_Socket_HighDensity_MountingHoles -> _Custom:DE15_Socket_HighDensity_MountingHoles
Connections:
- net iCE40-SDI: now also J21.3 (Pin_3); no longer J21.2 (Pin_2)
- net iCE40-SDO: now also J21.2 (Pin_2); no longer J21.3 (Pin_3)
Changed lines of the file:
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@@
 		(date "2024-09-17")
 		(rev "B")
-		(comment 1 "Changed to RP2352A to remove one of the flash ic's")
+		(comment 1 "Swaped SDI and SDO so you can use a straight through cable.")
+		(comment 2 "Changed to RP2352A to remove one of the flash ic's")
 	)
 	(text "VGA_GREEN_SHIELD"
@@
 	)
 	(junction
+		(at 129.54 312.42)
+		(diameter 0)
+		(color 0 0 0 0)
+	)
+	(junction
 		(at 726.44 63.5)
 		(diameter 0)
@@
 	)
 	(junction
-		(at 129.54 314.96)
-		(diameter 0)
-		(color 0 0 0 0)
-	)
-	(junction
 		(at 614.68 340.36)
 		(diameter 0)
@@
 	)
 	(junction
-		(at 726.44 137.16)
+		(at 137.16 314.96)
 		(diameter 0)
 		(color 0 0 0 0)
 	)
 	(junction
-		(at 137.16 317.5)
+		(at 726.44 137.16)
 		(diameter 0)
 		(color 0 0 0 0)
@@
 	(wire
 		(pts
-			(xy 137.16 317.5) (xy 182.88 317.5)
+			(xy 160.02 317.5) (xy 182.88 317.5)
 		)
 		(stroke
@@
 	(wire
 		(pts
-			(xy 129.54 314.96) (xy 182.88 314.96)
+			(xy 104.14 314.96) (xy 137.16 314.96)
 		)
 		(stroke
@@
 	(wire
 		(pts
-			(xy 137.16 312.42) (xy 137.16 317.5)
+			(xy 160.02 312.42) (xy 160.02 317.5)
 		)
 		(stroke
@@
 	(wire
 		(pts
+			(xy 137.16 314.96) (xy 182.88 314.96)
+		)
+		(stroke
+			(width 0)
+			(type default)
+		)
+	)
+	(wire
+		(pts
 			(xy 523.24 317.5) (xy 525.78 317.5)
 		)
@@
 	(wire
 		(pts
-			(xy 137.16 317.5) (xy 137.16 350.52)
+			(xy 408.94 414.02) (xy 408.94 378.46)
 		)
 		(stroke
@@
 	(wire
 		(pts
-			(xy 408.94 414.02) (xy 408.94 378.46)
+			(xy 571.5 180.34) (xy 584.2 180.34)
 		)
 		(stroke
@@
 	(wire
 		(pts
-			(xy 571.5 180.34) (xy 584.2 180.34)
+			(xy 337.82 203.2) (xy 330.2 203.2)
 		)
 		(stroke
@@
 	(wire
 		(pts
-			(xy 337.82 203.2) (xy 330.2 203.2)
+			(xy 589.28 330.2) (xy 601.98 330.2)
 		)
 		(stroke
@@
 	(wire
 		(pts
-			(xy 589.28 330.2) (xy 601.98 330.2)
+			(xy 134.62 375.92) (xy 142.24 375.92)
 		)
 		(stroke
@@
 	(wire
 		(pts
-			(xy 134.62 375.92) (xy 142.24 375.92)
+			(xy 116.84 495.3) (xy 111.76 495.3)
 		)
 		(stroke
@@
 	(wire
 		(pts
-			(xy 116.84 495.3) (xy 111.76 495.3)
+			(xy 129.54 312.42) (xy 160.02 312.42)
 		)
 		(stroke
@@
 	(wire
 		(pts
+			(xy 137.16 314.96) (xy 137.16 350.52)
+		)
+		(stroke
+			(width 0)
+			(type default)
+		)
+	)
+	(wire
+		(pts
 			(xy 127 502.92) (xy 127 508)
 		)
@@
 	(wire
 		(pts
+			(xy 129.54 312.42) (xy 129.54 347.98)
+		)
+		(stroke
+			(width 0)
+			(type default)
+		)
+	)
+	(wire
+		(pts
 			(xy 320.04 91.44) (xy 330.2 91.44)
 		)
@@
 	(wire
 		(pts
-			(xy 104.14 314.96) (xy 129.54 314.96)
-		)
-		(stroke
-			(width 0)
-			(type default)
-		)
-	)
-	(wire
-		(pts
 			(xy 208.28 116.84) (xy 185.42 116.84)
 		)
@@
 	(wire
 		(pts
-			(xy 129.54 347.98) (xy 129.54 314.96)
-		)
-		(stroke
-			(width 0)
-			(type default)
-		)
-	)
-	(wire
-		(pts
 			(xy 614.68 137.16) (xy 614.68 144.78)
 		)
@@
 	(wire
 		(pts
-			(xy 104.14 312.42) (xy 137.16 312.42)
+			(xy 104.14 312.42) (xy 129.54 312.42)
 		)
 		(stroke
@@
 		)
 	)
-	(label "iCE40-SDO"
-		(at 96.52 350.52 0)
-		(effects
-			(font
-				(size 1.524 1.524)
-			)
-			(justify left bottom)
-		)
-	)
 	(label "5v0.DC0"
 		(at 762 198.12 0)
@@
 		)
 	)
+	(label "iCE40-SDI"
+		(at 96.52 350.52 0)
+		(effects
+			(font
+				(size 1.524 1.524)
+			)
+			(justify left bottom)
+		)
+	)
 	(label "5v0.DB0"
 		(at 701.04 129.54 0)
@@
 		)
 	)
+	(label "iCE40-SDO"
+		(at 96.52 347.98 0)
+		(effects
+			(font
+				(size 1.524 1.524)
+			)
+			(justify left bottom)
+		)
+	)
 	(label "3v3.DE3"
 		(at 574.04 342.9 0)
@@
 		)
 	)
-	(label "iCE40-SDI"
-		(at 96.52 347.98 0)
-		(effects
-			(font
-				(size 1.524 1.524)
-			)
-			(justify left bottom)
-		)
-	)
 	(label "5v0.DE2"
 		(at 762 340.36 0)
@@
 	)
 	(symbol
-		(lib_id "Connector:DE15_Socket_HighDensity_MountingHoles")
+		(lib_id "_Custom:DE15_Socket_HighDensity_MountingHoles")
 		(at 248.92 441.96 0)
 		(unit 1)
@@
 			)
 		)
-		(property "Footprint" "SamacSys_Parts:117345301"
+		(property "Footprint" "_Custom:DSUB-15"
 			(at 224.79 431.8 0)
 			(hide yes)
