File: DaveFPGA/KiCad/Ice40hx4k_tq144.kicad_pcb (KiCad board)
At the start: 2 copper layers, 99.1 x 99.1 mm, 229 parts, among them J1 +5V, J2 +3V3, J21 PROGRAM, J22 USB_B_Micro, J3 SWD, J4 VGA, J9 2354 BOOT SEL, U1 LD1117S33TR_SOT223, U10 74CBTD3861, U11 LSF0108PW, U12 LSF0108PW, U13 LSF0108PW, U14 LSF0108PW, U15 74CBTD3861, U16 iCE40HX4K-TQ144, U18 TLV74311PDBVR, U19 RP2354A-QFN60, U2 MIC5504-1.2YM5, U3 W25Q16JVSSIQ, U5 LSF0108PW, U6 74CBTD3861, U7 74CBTD3861, U8 74CBTD3861, U9 74CBTD3861, Y1 12MHz

Commit message: - Changed crystal load capacitors from 12pf to 10pf.  This results in a clock frequency very slightly high instead of slightly low.
Parts:
- C25, C26: value 12pf -> 10pf
Changed lines of the file:
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@@
 			)
 		)
-		(property "Value" "12pf"
+		(property "Value" "10pf"
 			(at 0 1.43 0)
 			(layer "F.SilkS")
@@
 			)
 		)
-		(property "Value" "12pf"
+		(property "Value" "10pf"
 			(at 0 1.43 0)
 			(layer "F.SilkS")
@@
 		(layer "F.Cu")
 		(hatch none 0.1)
-		(priority 30001)
+		(priority 30035)
 		(attr
 			(teardrop
@@
 		(layer "F.Cu")
 		(hatch none 0.1)
-		(priority 31119)
+		(priority 30729)
 		(attr
 			(teardrop
@@
 		(polygon
 			(pts
-				(xy 75.016328 109.520562) (xy 75.193104 109.697338) (xy 74.759827 109.652517) (xy 75.353613 109.360053)
-				(xy 74.759827 109.652517)
+				(xy 75.688079 109.202363) (xy 75.511303 109.025587) (xy 74.972894 109.283475) (xy 75.10401 109.609656)
+				(xy 75.430191 109.740772)
 			)
 		)
@@
 		(layer "F.Cu")
 		(hatch none 0.1)
-		(priority 30728)
+		(priority 31119)
 		(attr
 			(teardrop
@@
 		(polygon
 			(pts
-				(xy 75.688079 109.202363) (xy 75.511303 109.025587) (xy 74.972894 109.283475) (xy 75.10401 109.609656)
-				(xy 75.430191 109.740772)
+				(xy 75.016328 109.520562) (xy 75.193104 109.697338) (xy 74.759827 109.652517) (xy 75.353613 109.360053)
+				(xy 74.759827 109.652517)
 			)
 		)
@@
 		(layer "F.Cu")
 		(hatch none 0.1)
-		(priority 30729)
+		(priority 30728)
 		(attr
 			(teardrop
@@
 		(layer "F.Cu")
 		(hatch none 0.1)
-		(priority 30005)
+		(priority 30128)
 		(attr
 			(teardrop
@@
 		(layer "F.Cu")
 		(hatch none 0.1)
-		(priority 30002)
+		(priority 30038)
 		(attr
 			(teardrop
@@
 		(layer "F.Cu")
 		(hatch none 0.1)
-		(priority 30003)
+		(priority 30039)
 		(attr
 			(teardrop
@@
 		(layer "F.Cu")
 		(hatch none 0.1)
-		(priority 30004)
+		(priority 30040)
 		(attr
 			(teardrop
@@
 		(layer "F.Cu")
 		(hatch none 0.1)
-		(priority 30731)
+		(priority 30756)
 		(attr
 			(teardrop
@@
 		(polygon
 			(pts
-				(xy 79.54553 111.468754) (xy 79.368754 111.64553) (xy 79.626642 112.183939) (xy 79.952823 112.052823)
-				(xy 80.083939 111.726642)
+				(xy 80.311611 112.588388) (xy 80.488388 112.411611) (xy 80.273358 111.916061) (xy 79.947177 112.047177)
+				(xy 79.816061 112.373358)
 			)
 		)
@@
 		(layer "F.Cu")
 		(hatch none 0.1)
-		(priority 31120)
+		(priority 30731)
 		(attr
 			(teardrop
@@
 		(polygon
 			(pts
-				(xy 80.036271 111.959495) (xy 79.859495 112.136271) (xy 79.602994 112.095684) (xy 80.19678 112.29678)
-				(xy 79.602994 112.095684)
+				(xy 79.54553 111.468754) (xy 79.368754 111.64553) (xy 79.626642 112.183939) (xy 79.952823 112.052823)
+				(xy 80.083939 111.726642)
 			)
 		)
@@
 		(layer "F.Cu")
 		(hatch none 0.1)
-		(priority 30756)
+		(priority 31120)
 		(attr
 			(teardrop
@@
 		(polygon
 			(pts
-				(xy 80.311611 112.588388) (xy 80.488388 112.411611) (xy 80.273358 111.916061) (xy 79.947177 112.047177)
-				(xy 79.816061 112.373358)
+				(xy 80.036271 111.959495) (xy 79.859495 112.136271) (xy 79.602994 112.095684) (xy 80.19678 112.29678)
+				(xy 79.602994 112.095684)
 			)
 		)
@@
 		(polygon
 			(pts
-				(xy 82.15447 112.031246) (xy 82.331246 111.85447) (xy 82.073358 111.316061) (xy 81.747177 111.447177)
-				(xy 81.616061 111.773358)
+				(xy 81.34553 110.868754) (xy 81.168754 111.04553) (xy 81.426642 111.583939) (xy 81.752823 111.452823)
+				(xy 81.883939 111.126642)
 			)
 		)
@@
 		(polygon
 			(pts
-				(xy 81.34553 110.868754) (xy 81.168754 111.04553) (xy 81.426642 111.583939) (xy 81.752823 111.452823)
-				(xy 81.883939 111.126642)
+				(xy 82.15447 112.031246) (xy 82.331246 111.85447) (xy 82.073358 111.316061) (xy 81.747177 111.447177)
+				(xy 81.616061 111.773358)
 			)
 		)
@@
 		(layer "F.Cu")
 		(hatch none 0.1)
-		(priority 30000)
+		(priority 30028)
 		(attr
 			(teardrop
@@
 		(layer "B.Cu")
 		(hatch none 0.1)
-		(priority 30001)
+		(priority 30017)
 		(attr
 			(teardrop
@@
 		(layer "B.Cu")
 		(hatch none 0.1)
-		(priority 30000)
+		(priority 30016)
 		(attr
 			(teardrop
