File: DaveFPGA/KiCad/Ice40hx4k_tq144.kicad_sch (KiCad schematic)
At the start: 229 parts, among them J1 +5V, J2 +3V3, J21 PROGRAM, J22 USB_B_Micro, J3 SWD, J4 VGA, J9 2354 BOOT SEL, U1 LD1117S33TR_SOT223, U10 74CBTD3861, U11 LSF0108PW, U12 LSF0108PW, U13 LSF0108PW, U14 LSF0108PW, U15 74CBTD3861, U16 iCE40HX4K-TQ144, U18 TLV74311PDBVR, U19 RP2354A-QFN60, U2 MIC5504-1.2YM5, U3 W25Q16JVSSIQ, U5 LSF0108PW, U6 74CBTD3861, U7 74CBTD3861, U8 74CBTD3861, U9 74CBTD3861, Y1 12MHz

Commit message: - Changed crystal load capacitors from 12pf to 10pf.  This results in a clock frequency very slightly high instead of slightly low.
Parts:
- C25, C26: value 12pf -> 10pf
Changed lines of the file:
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@@
 			)
 		)
-		(property "Value" "12pf"
+		(property "Value" "10pf"
 			(at 66.04 172.72 90)
 			(show_name no)
@@
 			)
 		)
-		(property "Value" "12pf"
+		(property "Value" "10pf"
 			(at 66.04 160.02 90)
 			(show_name no)
