File: DaveFPGA/KiCad/Ice40hx4k_tq144/Ice40hx4k_tq144.kicad_pcb (KiCad board)
At the start: 2 copper layers, 99.1 x 99.1 mm, 229 parts, among them J1 +5V, J2 +3V3, J21 PROGRAM, J22 USB_B_Micro, J3 SWD, J4 VGA, J9 2354 BOOT SEL, U1 LD1117S33TR_SOT223, U10 74CBTD3861, U11 LSF0108PW, U12 LSF0108PW, U13 LSF0108PW, U14 LSF0108PW, U15 74CBTD3861, U16 iCE40HX4K-TQ144, U18 TLV74311PDBVR, U19 RP2354A-QFN60, U2 MIC5504-1.2YM5, U3 W25Q16JVSSIQ, U5 LSF0108PW, U6 74CBTD3861, U7 74CBTD3861, U8 74CBTD3861, U9 74CBTD3861, Y1 12MHz

Commit message: - Created a new iCE40hx1k_vq100 based board with a rp2354 incorporated. I want to try a workflow of using SWD to flash the pico 2 and upload directly rather than flashing a seperate spi flash ic.
Parts:
- CDone1, Power1: footprint SamacSys_Parts:LEDC2012X90N -> LED_SMD:LED_0805_2012Metric
- J22: footprint Dave Footprints:USB_Micro-B_Amphenol_10103594-0001LF_Horizontal -> _Custom:USB_Micro-B_Amphenol_10103594-0001LF_Horizontal
- R51: value 1k -> 2k2
- U16: footprint SamacSys_Parts:QFP50P2200X2200X160-144N -> Package_QFP:LQFP-144_20x20mm_P0.5mm
- U3: footprint Dave Footprints:SOIC-8_5.23x5.23mm_P1.27mm -> Package_SO:SOIC-8_5.3x5.3mm_P1.27mm

Commit message: - Updated to kicad 10.0.6
Parts:
- U3: value W25Q16JVSSIQ -> W25Q16JVSS
Changed lines of the file:
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@@
 			)
 		)
-		(property "Value" "W25Q16JVSSIQ"
+		(property "Value" "W25Q16JVSS"
 			(at 0 3.6 0)
 			(layer "F.Fab")
@@
 			)
 		)
-		(property ki_fp_filters "SOIC*5.23x5.23mm*P1.27mm*")
+		(property ki_fp_filters "*SOIC*5.3x5.3mm*P1.27mm*")
 		(sheetname "/")
 		(sheetfile "Ice40hx4k_tq144.kicad_sch")
@@
 			(unit
 				(name "A")
-				(pins "8" "4" "1" "6" "5" "2" "3" "7")
+				(pins "1" "6" "5" "2" "3" "7" "8" "4")
 			)
 		)
@@
 			(roundrect_rratio 0.25)
 			(net "/iCE40-SDI")
-			(pinfunction "DO(IO1)_2")
+			(pinfunction "DO/IO_{1}_2")
 			(pintype "bidirectional")
 		)
@@
 			(layers "F.Cu" "F.Mask" "F.Paste")
 			(roundrect_rratio 0.25)
-			(net "Net-(U3-~{HOLD}(IO3))")
-			(pinfunction "~{WP}(IO2)_3")
+			(net "Net-(U3-~{HOLD}{slash}~{RESET}{slash}IO_{3})")
+			(pinfunction "~{WP}/IO_{2}_3")
 			(pintype "bidirectional")
 		)
@@
 			(roundrect_rratio 0.25)
 			(net "/iCE40-SDO")
-			(pinfunction "DI(IO0)_5")
+			(pinfunction "DI/IO_{0}_5")
 			(pintype "bidirectional")
 		)
@@
 			(layers "F.Cu" "F.Mask" "F.Paste")
 			(roundrect_rratio 0.25)
-			(net "Net-(U3-~{HOLD}(IO3))")
-			(pinfunction "~{HOLD}(IO3)_7")
+			(net "Net-(U3-~{HOLD}{slash}~{RESET}{slash}IO_{3})")
+			(pinfunction "~{HOLD}/~{RESET}/IO_{3}_7")
 			(pintype "bidirectional")
 		)
@@
 			(layers "F.Cu" "F.Mask" "F.Paste")
 			(roundrect_rratio 0.25)
-			(net "Net-(U3-~{HOLD}(IO3))")
+			(net "Net-(U3-~{HOLD}{slash}~{RESET}{slash}IO_{3})")
 			(pintype "passive")
 			(teardrops
@@
 			(unit
 				(name "A")
-				(pins "2" "1")
+				(pins "1" "2")
 			)
 		)
@@
 		(width 0.25)
 		(layer "F.Cu")
-		(net "Net-(U3-~{HOLD}(IO3))")
+		(net "Net-(U3-~{HOLD}{slash}~{RESET}{slash}IO_{3})")
 	)
 	(segment
@@
 		(width 0.25)
 		(layer "F.Cu")
-		(net "Net-(U3-~{HOLD}(IO3))")
+		(net "Net-(U3-~{HOLD}{slash}~{RESET}{slash}IO_{3})")
 	)
 	(segment
@@
 		(width 0.25)
 		(layer "F.Cu")
-		(net "Net-(U3-~{HOLD}(IO3))")
+		(net "Net-(U3-~{HOLD}{slash}~{RESET}{slash}IO_{3})")
 	)
 	(segment
@@
 		(width 0.25)
 		(layer "F.Cu")
-		(net "Net-(U3-~{HOLD}(IO3))")
+		(net "Net-(U3-~{HOLD}{slash}~{RESET}{slash}IO_{3})")
 	)
 	(via
@@
 			(prefer_zone_connections yes)
 		)
-		(net "Net-(U3-~{HOLD}(IO3))")
+		(net "Net-(U3-~{HOLD}{slash}~{RESET}{slash}IO_{3})")
 	)
 	(via
@@
 			(prefer_zone_connections yes)
 		)
-		(net "Net-(U3-~{HOLD}(IO3))")
+		(net "Net-(U3-~{HOLD}{slash}~{RESET}{slash}IO_{3})")
 	)
 	(segment
@@
 		(width 0.25)
 		(layer "B.Cu")
-		(net "Net-(U3-~{HOLD}(IO3))")
+		(net "Net-(U3-~{HOLD}{slash}~{RESET}{slash}IO_{3})")
 	)
 	(segment
@@
 		(width 0.25)
 		(layer "B.Cu")
-		(net "Net-(U3-~{HOLD}(IO3))")
+		(net "Net-(U3-~{HOLD}{slash}~{RESET}{slash}IO_{3})")
 	)
 	(segment
@@
 	)
 	(zone
-		(net "Net-(U3-~{HOLD}(IO3))")
+		(net "Net-(U3-~{HOLD}{slash}~{RESET}{slash}IO_{3})")
 		(layer "F.Cu")
 		(hatch none 0.1)
-		(priority 30977)
+		(priority 30709)
 		(attr
 			(teardrop
@@
 		(polygon
 			(pts
-				(xy 75.016328 109.520562) (xy 75.193104 109.697338) (xy 74.759827 109.652517) (xy 75.353613 109.360053)
-				(xy 74.759827 109.652517)
+				(xy 75.688079 109.202363) (xy 75.511303 109.025587) (xy 74.972894 109.283475) (xy 75.10401 109.609656)
+				(xy 75.430191 109.740772)
 			)
 		)
 	)
 	(zone
-		(net "Net-(U3-~{HOLD}(IO3))")
+		(net "Net-(U3-~{HOLD}{slash}~{RESET}{slash}IO_{3})")
 		(layer "F.Cu")
 		(hatch none 0.1)
-		(priority 30708)
+		(priority 30977)
 		(attr
 			(teardrop
@@
 		(polygon
 			(pts
-				(xy 75.688079 109.202363) (xy 75.511303 109.025587) (xy 74.972894 109.283475) (xy 75.10401 109.609656)
-				(xy 75.430191 109.740772)
+				(xy 75.016328 109.520562) (xy 75.193104 109.697338) (xy 74.759827 109.652517) (xy 75.353613 109.360053)
+				(xy 74.759827 109.652517)
 			)
 		)
 	)
 	(zone
-		(net "Net-(U3-~{HOLD}(IO3))")
+		(net "Net-(U3-~{HOLD}{slash}~{RESET}{slash}IO_{3})")
 		(layer "F.Cu")
 		(hatch none 0.1)
-		(priority 30709)
+		(priority 30708)
 		(attr
 			(teardrop
@@
 		(layer "F.Cu")
 		(hatch none 0.1)
-		(priority 30737)
+		(priority 30711)
 		(attr
 			(teardrop
@@
 		(polygon
 			(pts
-				(xy 80.311611 112.588388) (xy 80.488388 112.411611) (xy 80.273358 111.916061) (xy 79.947177 112.047177)
-				(xy 79.816061 112.373358)
+				(xy 79.54553 111.468754) (xy 79.368754 111.64553) (xy 79.626642 112.183939) (xy 79.952823 112.052823)
+				(xy 80.083939 111.726642)
 			)
 		)
@@
 		(layer "F.Cu")
 		(hatch none 0.1)
-		(priority 30711)
+		(priority 30737)
 		(attr
 			(teardrop
@@
 		(polygon
 			(pts
-				(xy 79.54553 111.468754) (xy 79.368754 111.64553) (xy 79.626642 112.183939) (xy 79.952823 112.052823)
-				(xy 80.083939 111.726642)
+				(xy 80.311611 112.588388) (xy 80.488388 112.411611) (xy 80.273358 111.916061) (xy 79.947177 112.047177)
+				(xy 79.816061 112.373358)
 			)
 		)
@@
 		(layer "F.Cu")
 		(hatch none 0.1)
-		(priority 30712)
+		(priority 30979)
 		(attr
 			(teardrop
@@
 		(polygon
 			(pts
-				(xy 81.34553 110.868754) (xy 81.168754 111.04553) (xy 81.426642 111.583939) (xy 81.752823 111.452823)
-				(xy 81.883939 111.126642)
+				(xy 81.836271 111.359495) (xy 81.659495 111.536271) (xy 81.402994 111.495684) (xy 81.99678 111.69678)
+				(xy 81.402994 111.495684)
 			)
 		)
@@
 		(layer "F.Cu")
 		(hatch none 0.1)
-		(priority 30979)
+		(priority 30712)
 		(attr
 			(teardrop
@@
 		(polygon
 			(pts
-				(xy 81.836271 111.359495) (xy 81.659495 111.536271) (xy 81.402994 111.495684) (xy 81.99678 111.69678)
-				(xy 81.402994 111.495684)
+				(xy 81.34553 110.868754) (xy 81.168754 111.04553) (xy 81.426642 111.583939) (xy 81.752823 111.452823)
+				(xy 81.883939 111.126642)
 			)
 		)
@@
 	)
 	(zone
-		(net "Net-(U3-~{HOLD}(IO3))")
+		(net "Net-(U3-~{HOLD}{slash}~{RESET}{slash}IO_{3})")
 		(layer "F.Cu")
 		(hatch none 0.1)
@@
 	)
 	(zone
-		(net "Net-(U3-~{HOLD}(IO3))")
+		(net "Net-(U3-~{HOLD}{slash}~{RESET}{slash}IO_{3})")
 		(layer "F.Cu")
 		(hatch none 0.1)
@@
 	)
 	(zone
-		(net "Net-(U3-~{HOLD}(IO3))")
+		(net "Net-(U3-~{HOLD}{slash}~{RESET}{slash}IO_{3})")
 		(layer "B.Cu")
 		(hatch none 0.1)
@@
 	)
 	(zone
-		(net "Net-(U3-~{HOLD}(IO3))")
+		(net "Net-(U3-~{HOLD}{slash}~{RESET}{slash}IO_{3})")
 		(layer "B.Cu")
 		(hatch none 0.1)
