File: DaveFPGA/KiCad/Ice40hx4k_tq144/Ice40hx4k_tq144.kicad_sch (KiCad schematic)
At the start: 229 parts, among them J1 +5V, J2 +3V3, J21 PROGRAM, J22 USB_B_Micro, J3 SWD, J4 VGA, J9 2354 BOOT SEL, U1 LD1117S33TR_SOT223, U10 74CBTD3861, U11 LSF0108PW, U12 LSF0108PW, U13 LSF0108PW, U14 LSF0108PW, U15 74CBTD3861, U16 iCE40HX4K-TQ144, U18 TLV74311PDBVR, U19 RP2354A-QFN60, U2 MIC5504-1.2YM5, U3 W25Q16JVSSIQ, U5 LSF0108PW, U6 74CBTD3861, U7 74CBTD3861, U8 74CBTD3861, U9 74CBTD3861, Y1 12MHz

Commit message: - Created a new iCE40hx1k_vq100 based board with a rp2354 incorporated. I want to try a workflow of using SWD to flash the pico 2 and upload directly rather than flashing a seperate spi flash ic.
Parts:
- CDone1, Power1: footprint SamacSys_Parts:LEDC2012X90N -> LED_SMD:LED_0805_2012Metric
- J22: footprint Dave Footprints:USB_Micro-B_Amphenol_10103594-0001LF_Horizontal -> _Custom:USB_Micro-B_Amphenol_10103594-0001LF_Horizontal
- R50: now not fitted
- R51: value 1k -> 2k2
- U16: footprint SamacSys_Parts:QFP50P2200X2200X160-144N -> Package_QFP:LQFP-144_20x20mm_P0.5mm; symbol Dave:iCE40HX4K-TQ144 -> _Custom:iCE40HX4K-TQ144
- U3: footprint Dave Footprints:SOIC-8_5.23x5.23mm_P1.27mm -> Package_SO:SOIC-8_5.3x5.3mm_P1.27mm
Other:
- note added: "CSn0"
- note added: "RX0"
- note added: "SCK0"
- note added: "TX0"
Changed lines of the file:
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@@
 		)
 	)
+	(text "RX0"
+		(exclude_from_sim no)
+		(at 185.42 139.7 0)
+		(effects
+			(font
+				(size 1.27 1.27)
+			)
+		)
+	)
+	(text "SCK0"
+		(exclude_from_sim no)
+		(at 185.42 144.78 0)
+		(effects
+			(font
+				(size 1.27 1.27)
+			)
+		)
+	)
 	(text "VGA_SYNC_RETURN"
 		(exclude_from_sim no)
@@
 		)
 	)
+	(text "TX0"
+		(exclude_from_sim no)
+		(at 185.42 137.16 0)
+		(effects
+			(font
+				(size 1.27 1.27)
+			)
+		)
+	)
 	(text "VGA_RED_SHIELD"
 		(exclude_from_sim no)
@@
 		)
 	)
+	(text "CSn0"
+		(exclude_from_sim no)
+		(at 185.42 142.24 0)
+		(effects
+			(font
+				(size 1.27 1.27)
+			)
+		)
+	)
 	(text "VGA_ID_BIT0"
 		(exclude_from_sim no)
@@
 	)
 	(symbol
-		(lib_id "Dave:iCE40HX4K-TQ144")
+		(lib_id "_Custom:iCE40HX4K-TQ144")
 		(at 205.74 312.42 0)
 		(unit 5)
@@
 			)
 		)
-		(property "Footprint" "SamacSys_Parts:QFP50P2200X2200X160-144N"
-			(at 141.732 200.914 0)
+		(property "Footprint" "Package_QFP:LQFP-144_20x20mm_P0.5mm"
+			(at 185.42 263.398 0)
 			(hide yes)
 			(show_name no)
@@
 		)
 		(property "Description" "FPGA - Field Programmable Gate Array"
-			(at 155.702 195.834 0)
+			(at 205.994 259.334 0)
 			(hide yes)
 			(show_name no)
@@
 			)
 		)
-		(property "Footprint" "SamacSys_Parts:LEDC2012X90N"
+		(property "Footprint" "LED_SMD:LED_0805_2012Metric"
 			(at 167.64 364.49 0)
 			(hide yes)
@@
 			)
 		)
-		(property "Footprint" "Dave Footprints:SOIC-8_5.23x5.23mm_P1.27mm"
+		(property "Footprint" "Package_SO:SOIC-8_5.3x5.3mm_P1.27mm"
 			(at 93.218 344.17 0)
 			(hide yes)
@@
 			)
 		)
-		(property "Value" "1k"
+		(property "Value" "2k2"
 			(at 66.04 137.16 90)
 			(show_name no)
@@
 			)
 		)
-		(property "Footprint" "SamacSys_Parts:LEDC2012X90N"
+		(property "Footprint" "LED_SMD:LED_0805_2012Metric"
 			(at 99.06 485.14 0)
 			(hide yes)
@@
 	)
 	(symbol
-		(lib_id "Dave:iCE40HX4K-TQ144")
+		(lib_id "_Custom:iCE40HX4K-TQ144")
 		(at 548.64 350.52 0)
 		(unit 3)
@@
 			)
 		)
-		(property "Footprint" "SamacSys_Parts:QFP50P2200X2200X160-144N"
-			(at 484.632 239.014 0)
+		(property "Footprint" "Package_QFP:LQFP-144_20x20mm_P0.5mm"
+			(at 528.32 301.498 0)
 			(hide yes)
 			(show_name no)
@@
 		)
 		(property "Description" "FPGA - Field Programmable Gate Array"
-			(at 498.602 233.934 0)
+			(at 548.894 297.434 0)
 			(hide yes)
 			(show_name no)
@@
 	)
 	(symbol
-		(lib_id "Dave:iCE40HX4K-TQ144")
+		(lib_id "_Custom:iCE40HX4K-TQ144")
 		(at 439.42 350.52 0)
 		(mirror y)
@@
 			)
 		)
-		(property "Footprint" "SamacSys_Parts:QFP50P2200X2200X160-144N"
-			(at 503.428 239.014 0)
+		(property "Footprint" "Package_QFP:LQFP-144_20x20mm_P0.5mm"
+			(at 459.74 301.498 0)
 			(hide yes)
 			(show_name no)
@@
 		)
 		(property "Description" "FPGA - Field Programmable Gate Array"
-			(at 489.458 233.934 0)
+			(at 439.166 297.434 0)
 			(hide yes)
 			(show_name no)
@@
 		(property "Value" "PWR_FLAG"
 			(at 109.5193 105.6368 0)
+			(hide yes)
 			(show_name no)
 			(do_not_autoplace no)
@@
 			)
 		)
-		(property "Footprint" "Dave Footprints:USB_Micro-B_Amphenol_10103594-0001LF_Horizontal"
+		(property "Footprint" "_Custom:USB_Micro-B_Amphenol_10103594-0001LF_Horizontal"
 			(at 217.17 110.49 0)
 			(hide yes)
@@
 	)
 	(symbol
-		(lib_id "Dave:iCE40HX4K-TQ144")
+		(lib_id "_Custom:iCE40HX4K-TQ144")
 		(at 439.42 157.48 0)
 		(mirror y)
@@
 			)
 		)
-		(property "Footprint" "SamacSys_Parts:QFP50P2200X2200X160-144N"
-			(at 503.428 45.974 0)
+		(property "Footprint" "Package_QFP:LQFP-144_20x20mm_P0.5mm"
+			(at 459.74 108.458 0)
 			(hide yes)
 			(show_name no)
@@
 		)
 		(property "Description" "FPGA - Field Programmable Gate Array"
-			(at 489.458 40.894 0)
+			(at 439.166 104.394 0)
 			(hide yes)
 			(show_name no)
@@
 	)
 	(symbol
-		(lib_id "Dave:iCE40HX4K-TQ144")
+		(lib_id "_Custom:iCE40HX4K-TQ144")
 		(at 548.64 157.48 0)
 		(unit 1)
@@
 			)
 		)
-		(property "Footprint" "SamacSys_Parts:QFP50P2200X2200X160-144N"
-			(at 484.632 45.974 0)
+		(property "Footprint" "Package_QFP:LQFP-144_20x20mm_P0.5mm"
+			(at 528.32 108.458 0)
 			(hide yes)
 			(show_name no)
@@
 		)
 		(property "Description" "FPGA - Field Programmable Gate Array"
-			(at 498.602 40.894 0)
+			(at 548.894 104.394 0)
 			(hide yes)
 			(show_name no)
@@
 		(on_board yes)
 		(in_pos_files yes)
-		(dnp no)
+		(dnp yes)
 		(property "Reference" "R50"
 			(at 71.7366 132.118 90)

Commit message: - Updated to kicad 10.0.6
Parts:
- CDone1: symbol Dave:LED -> Device:LED_Small_Filled
- U3: value W25Q16JVSSIQ -> W25Q16JVSS; symbol Dave:W25Q16JVSSIQ -> Memory_Flash:W25Q16JVSS
Other:
- moved on the sheet: U3
Changed lines of the file:
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@@
 	)
 	(junction
-		(at 167.64 355.6)
-		(diameter 0)
-		(color 0 0 0 0)
-	)
-	(junction
 		(at 127 106.68)
 		(diameter 0)
@@
 	)
 	(junction
+		(at 167.64 355.6)
+		(diameter 0)
+		(color 0 0 0 0)
+	)
+	(junction
 		(at 111.76 495.3)
 		(diameter 0)
@@
 	(wire
 		(pts
-			(xy 167.64 368.3) (xy 167.64 370.84)
-		)
-		(stroke
-			(width 0)
-			(type default)
-		)
-	)
-	(wire
-		(pts
 			(xy 502.92 327.66) (xy 508 327.66)
 		)
@@
 	(wire
 		(pts
-			(xy 167.64 355.6) (xy 167.64 360.68)
-		)
-		(stroke
-			(width 0)
-			(type default)
-		)
-	)
-	(wire
-		(pts
 			(xy 134.62 365.76) (xy 134.62 368.3)
 		)
@@
 	(wire
 		(pts
+			(xy 167.64 355.6) (xy 167.64 360.68)
+		)
+		(stroke
+			(width 0)
+			(type default)
+		)
+	)
+	(wire
+		(pts
 			(xy 167.64 353.06) (xy 167.64 355.6)
 		)
@@
 	(wire
 		(pts
+			(xy 167.64 365.76) (xy 167.64 370.84)
+		)
+		(stroke
+			(width 0)
+			(type default)
+		)
+	)
+	(wire
+		(pts
 			(xy 614.68 162.56) (xy 607.06 162.56)
 		)
@@
 	)
 	(symbol
-		(lib_id "Dave:LED")
-		(at 167.64 365.76 270)
+		(lib_id "Device:LED_Small_Filled")
+		(at 167.64 363.22 90)
 		(unit 1)
 		(body_style 1)
@@
 		(dnp no)
 		(property "Reference" "CDone1"
-			(at 170.18 369.57 0)
+			(at 165.1 359.41 0)
 			(hide yes)
 			(show_name no)
@@
 		)
 		(property "Value" "DONE"
-			(at 170.9631 367.2956 0)
+			(at 170.18 360.68 0)
 			(show_name no)
 			(do_not_autoplace no)
@@
 		)
 		(property "Description" "Light emitting diode, filled shape"
-			(at 160.274 366.014 0)
+			(at 175.006 362.966 0)
 			(hide yes)
 			(show_name no)
@@
 		)
 		(property "Note" ""
-			(at 167.64 365.76 0)
+			(at 167.64 363.22 0)
 			(hide yes)
 			(show_name no)
@@
 		)
 		(property "Voltage" ""
-			(at 167.64 365.76 0)
+			(at 167.64 363.22 0)
 			(hide yes)
 			(show_name no)
@@
 		)
 		(property "class" ""
-			(at 167.64 365.76 0)
+			(at 167.64 363.22 0)
 			(hide yes)
 			(show_name no)
@@
 	)
 	(symbol
-		(lib_id "Dave:W25Q16JVSSIQ")
+		(lib_id "Memory_Flash:W25Q16JVSS")
 		(at 93.98 314.96 0)
+		(mirror y)
 		(unit 1)
 		(body_style 1)
@@
 		(dnp no)
 		(property "Reference" "U3"
-			(at 90.2832 303.0417 0)
+			(at 97.6768 303.0417 0)
 			(show_name no)
 			(do_not_autoplace no)
@@
 			)
 		)
-		(property "Value" "W25Q16JVSSIQ"
-			(at 88.9 307.34 90)
+		(property "Value" "W25Q16JVSS"
+			(at 99.06 307.34 90)
 			(show_name no)
 			(do_not_autoplace no)
@@
 		)
 		(property "Footprint" "Package_SO:SOIC-8_5.3x5.3mm_P1.27mm"
-			(at 93.218 344.17 0)
+			(at 94.742 344.17 0)
 			(hide yes)
 			(show_name no)
@@
 		)
 		(property "Datasheet" "https://au.mouser.com/datasheet/2/949/w25q16jv_spi_revg_03222018_plus-1489727.pdf"
-			(at 93.472 348.488 0)
+			(at 94.488 348.488 0)
 			(hide yes)
 			(show_name no)
