File: DaveFPGA/KiCad/Ice40hx1k_vq100/Ice40hx1k_vq100.kicad_pcb (KiCad board)
At the start: 2 copper layers, 99.1 x 99.1 mm, 153 parts, among them J1 +5V, J10 VGA, J2 +3v3, J3 USB_B_Micro, J4 VGA, J5 SWD, U1 LD1117S33TR_SOT223, U10 74CBTD3861, U11 LSF0108PW, U12 74CBTD3861, U2 MIC5504-1.2YM5, U3 iCE40HX4K-TQ144, U4 TLV74311PDBVR, U5 RP2354A-QFN60, U6 LSF0108PW, U7 74CBTD3861, U8 74CBTD3861, U9 LSF0108PW, Y1 12MHz

Commit message: - Created a new FPGA prototyping board based around the iCE40hx1k and the rp2354.
Parts:
- R22: moved to F.Cu
- U3: value iCE40HX4K-TQ144 -> iCE40HX1K-VQ100
- moved R22 18.2 mm to (99.7, 61.2), turned to 90 degrees
- moved R2 1.57 mm to (97.0, 71.3), turned to -135 degrees
Connections:
- S1 pad 1: /~{3v3_RESET} -> Net-(U5-RUN)
Routing:
- net Net-(U5-RUN): track 5.06 -> 54.6 mm, vias 1 -> 2
- net /~{3v3_RESET}: track 117.3 -> 81.5 mm
- net +3V3: track 358.2 -> 368.4 mm
Other:
- board text added: "iCE40HX1K"
- board text removed: "iCE40hx1k"

Commit message: - Created design blocks for the RP2354 and iCE40hx1k_vq100
Parts:
- added C55: 100nf, Capacitor_SMD:C_0603_1608Metric, F.Cu at (100.4, 83.3)
- R11: moved to B.Cu
- moved R11 3.54 mm to (104.1, 85.5), turned to 45 degrees
Routing:
- net GND: track 118.7 -> 126.4 mm, vias 235 -> 239
- net /~{CS}: track 26.5 -> 24.8 mm, vias 0 -> 1
- net +3V3: track 368.4 -> 369.4 mm, vias 36 -> 37
